File: kicad/ble_door_sensor.kicad_pcb (KiCad board)
At the start: 4 copper layers, 20 x 61.5 mm, 41 parts, among them J1 Prog Header, J101 Conn_01x08, Q1 ALS-PT19, SW101 SW_Reed, SW102 SW_Push, T1 ToolingHole, T2 ToolingHole, T3 ToolingHole, U1 nRF52832-QFxx, U101 TMP100, U2 SHTC3, Y1 Crystal_GND24

Commit message: Move footprints to new library
Parts:
- SW101: footprint Library:reed_contact -> g-Sensors:reed_contact
- T1, T2, T3: footprint Library:JLCPCB_Mounting_hole -> g-Misc:JLCPCB_Mounting_hole

Commit message: Move sensors to a new different sheet
Parts:
- renumbered BT1 to BT201, C13 to C201, C101 to C202, C3 to C203, D101 to D201, H101 to H201, H102 to H202, J1 to J201, J101 to J202, Q1 to Q201, R102 to R201, R2 to R202, R101 to R203, R104 to R204, R105 to R205, R3 to R206, R1 to R207, SW101 to SW201, SW102 to SW202, T1 to T201, T2 to T202, T3 to T203, U2 to U201, U101 to U202
