File: kicad/sensors.kicad_sch (KiCad schematic)
At the start: 24 parts, among them J1 Prog Header, J101 Conn_01x08, Q1 ALS-PT19, SW101 SW_Reed, SW102 SW_Push, T1 ToolingHole, T2 ToolingHole, T3 ToolingHole, U101 TMP100, U2 SHTC3

Commit message: Move sensors to a new different sheet
Parts:
- removed H101, H102: MountingHole, MountingHole:MountingHole_2.2mm_M2, symbol Mechanical:MountingHole
- renumbered BT1 to BT201, C13 to C201, C101 to C202, C3 to C203, D101 to D201, J1 to J201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

Commit message: Add STM32WB55 based board
Parts:
- J202: now not fitted
